File: switcher/switcher.kicad_sch (KiCad schematic)
At the start: 11 parts

Commit message: Working version of python spicelib
Connections:
- net LOAD renamed load
Changed lines of the file:
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@@
 		)
 	)
-	(label "LOAD"
-		(at 245.11 88.9 180)
+	(global_label "source"
+		(shape input)
+		(at 55.88 73.66 180)
+		(fields_autoplaced yes)
 		(effects
 			(font
 				(size 1.27 1.27)
 			)
-			(justify right bottom)
+			(justify right)
+		)
+		(property "Intersheetrefs" "${INTERSHEET_REFS}"
+			(at 46.6053 73.66 0)
+			(hide yes)
+			(show_name no)
+			(do_not_autoplace no)
+			(effects
+				(font
+					(size 1.27 1.27)
+				)
+				(justify right)
+			)
 		)
 	)
-	(label "C1"
-		(at 152.4 91.44 180)
+	(global_label "load"
+		(shape input)
+		(at 245.11 88.9 0)
+		(fields_autoplaced yes)
 		(effects
 			(font
 				(size 1.27 1.27)
 			)
-			(justify right bottom)
+			(justify left)
+		)
+		(property "Intersheetrefs" "${INTERSHEET_REFS}"
+			(at 252.2074 88.9 0)
+			(hide yes)
+			(show_name no)
+			(do_not_autoplace no)
+			(effects
+				(font
+					(size 1.27 1.27)
+				)
+				(justify left)
+			)
 		)
 	)
-	(label "source"
-		(at 55.88 73.66 0)
+	(global_label "C1"
+		(shape input)
+		(at 152.4 91.44 0)
+		(fields_autoplaced yes)
 		(effects
 			(font
 				(size 1.27 1.27)
 			)
-			(justify left bottom)
+			(justify left)
+		)
+		(property "Intersheetrefs" "${INTERSHEET_REFS}"
+			(at 157.8647 91.44 0)
+			(hide yes)
+			(show_name no)
+			(do_not_autoplace no)
+			(effects
+				(font
+					(size 1.27 1.27)
+				)
+				(justify left)
+			)
 		)
 	)
@@
 			)
 		)
-		(property "Sim.Library" "/home/jtmadden/repos/jlab/switcher/cap.lib"
+		(property "Sim.Library" "/home/jtmadden/repos/jlab/shiny-train/cap.lib"
 			(at 132.08 96.52 0)
 			(hide yes)
